File: Skyfall_Avionic.kicad_pcb (KiCad board)
At the start: 2 copper layers, 50 x 80 mm, 83 parts, among them IC1 TPS62130ARGTR, IC2 TPS62130ARGTR, IC4 W25Q128JVEIM_TR, J1 M20-9720546, J2 USB4105-GF-A-060, J5 53261-0371, J6 53261-0271, J7 53261-0471, J8 53261-0671, Q2 SS8550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

Commit message: Minor PCB Changes
Routing:
- net LORA_CS: track 41.2 -> 49.8 mm
- net +3.3V: track 377.9 -> 380.4 mm, vias 20 -> 21
- net LORA_TXEN: track 80.7 -> 82.8 mm
- net LORA_RXEN: track 67.8 -> 69.8 mm
- net DIO2: track 71.6 -> 72.9 mm

Commit message: PCB Review
Parts:
- moved J7 0.08 mm to (165.8, 123.5)
Routing:
- net +3.3V: track 380.4 -> 379.3 mm

Commit message: Review
Parts:
- H1, H2, H3, H4: footprint MountingHole:MountingHole_2.7mm_M2.5_Pad -> MountingHole:MountingHole_2.7mm_M2.5_Pad_Via
- Q2, R14, R30, S1: moved to F.Cu
- moved Q2 28.5 mm to (167.8, 149.2), turned to 0 degrees
- moved R30 19.0 mm to (164.8, 148.1)
- moved LS1 8.28 mm to (156.0, 147.5), turned to 0 degrees
- moved R14 6.83 mm to (156.0, 100.0), turned to 180 degrees
- moved S1 2.34 mm to (157.7, 103.5)
- moved R2 0.70 mm to (159.6, 107.1)
- moved J7 0.11 mm to (165.7, 123.5)
Connections:
- H1 pad 1: unconnected-(H1-Pad1) -> GND
- H2 pad 1: unconnected-(H2-Pad1) -> GND
- H3 pad 1: unconnected-(H3-Pad1) -> GND
- H4 pad 1: unconnected-(H4-Pad1) -> GND
Routing:
- net Buzz: track 39.7 -> 59.0 mm, vias 3 -> 2
- net Net-(Q2-B): track 13.7 -> 2.51 mm
- net RESET: track 43.0 -> 48.8 mm, vias 1 -> 0
- net VIN: track 88.2 -> 86.2 mm
- net Net-(LS1--): track 6.39 -> 8.31 mm, vias 0 -> 1
- net +3.3V: track 379.3 -> 377.7 mm
- net GND: track 88.9 -> 87.8 mm
- net Servo: track 24.8 -> 25.7 mm
- net +5V: track 115.0 -> 114.3 mm
- net Net-(J2-CC2): track 4.72 -> 4.03 mm
- added copper zone on F.Cu, net VIN
